File: kicad pcb/EPD 3D G6/EPD 3D G6.kicad_sch (KiCad schematic)
At the start: 0 parts

Commit message: Update connector J_MAIN pinout: pin 2 CONN_DETECT loopback detect, gitignore KiCad backups/cache
Parts:
- added C1, C10, C13, C7: 100uF, symbol Device:C
- added C11, C12, C14, C15, C16, C17, C18, C19, C20, C3, C6, C8, C9: 100nF, symbol Device:C
- added C2, C4: 470uF, symbol Device:C
- added C5: 10uF, symbol Device:C
- added J1: J_ESP32_L, symbol Connector_Generic:Conn_01x10
- added J10: OLED, symbol Connector_Generic:Conn_01x04
- added J11: BAT+, symbol Connector:Conn_01x01_Pin
- added J12: BAT-, symbol Connector:Conn_01x01_Pin
- added J13: BOOST_IN+, symbol Connector:Conn_01x01_Pin
- added J14: BOOST_IN-, symbol Connector:Conn_01x01_Pin
- added J15, J16: BOOST_OUT+, symbol Connector:Conn_01x01_Pin
- added J2: J_ESP32_R, symbol Connector_Generic:Conn_01x10
- added J3: TMC2209_1_L, symbol Connector_Generic:Conn_01x08
- added J4: TMC2209_1_R, symbol Connector_Generic:Conn_01x08
- added J5: TMC2209_2_L, symbol Connector_Generic:Conn_01x08
- added J6: TMC2209_2_R, symbol Connector_Generic:Conn_01x08
- added J7: TMC2209_3_L, symbol Connector_Generic:Conn_01x08
- added J8: TMC2209_3_R, symbol Connector_Generic:Conn_01x08
- added J9: 20 PIN TO INSOLE, symbol Connector_Generic:Conn_02x10_Odd_Even
- added R1, R4, R6, R8: 1k, symbol Device:R
- added R10, R9: 100k, symbol Device:R
- added R2, R3, R5, R7: 10k, symbol Device:R
- added SW1: POWER_SWITCH, symbol Switch:SW_Push
- added SW2: SW_Push, symbol Switch:SW_Push
Connections:
- net 3V3: now also C12.1, C15.1, C5.2, C6.2, C9.1, J10.3V3 (Pin_2), J2.3V3 (Pin_8), J4.VDD (Pin_2), J6.VDD (Pin_2), J8.VDD (Pin_2)
- net 5V_SYS: now also C10.1, C11.1, C13.1, C14.1, C2.1, C3.1, C4.1, C7.1, C8.1, J15.+ (Pin_1), J2.5V (Pin_10), J4.VM (Pin_8), J6.VM (Pin_8), J8.VM (Pin_8)
- net ACT1_DIR: now also J2.GP19 (Pin_6), J3.DIR (Pin_8)
- net ACT1_STEP: now also J2.GP20 (Pin_7), J3.STEP (Pin_7)
- net ACT2_DIR: now also J2.GP14 (Pin_3), J5.DIR (Pin_8)
- net ACT2_STEP: now also J2.GP18 (Pin_5), J5.STEP (Pin_7)
- net ACT3_DIR: now also J1.RX (Pin_2), J7.DIR (Pin_8)
- net ACT3_STEP: now also J1.TX (Pin_1), J7.STEP (Pin_7)
- net CONN_DETECT: now also J1.GP5 (Pin_8), J9.2 (Pin_2)
- net FSR1_ADC: now also C16.1, J1.GP0 (Pin_3), R1.2
- net FSR2_ADC: now also C17.1, J1.GP1 (Pin_4), R4.2
- net FSR3_ADC: now also C18.1, J1.GP2 (Pin_5), R6.2
- net FSR4_ADC: now also C19.1, J1.GP3 (Pin_6), R8.2
- net MODE_BTN: now also J1.GP4 (Pin_7), SW2.1
- net OLED_SCL: now also J10.SCL (Pin_4), J2.GP15 (Pin_4)
- net OLED_SDA: now also J10.SDA (Pin_3), J2.GP9 (Pin_2)
- net STEPPER_ENN: now also J1.GP7 (Pin_10), J3.EN (Pin_1), J5.EN (Pin_1), J7.EN (Pin_1)
- net VBAT: now also C1.1, J13.+ (Pin_1), R9.1, SW1.2
- net VBAT_SENSE: now also C20.1, J1.GP6 (GP7), R10.2, R9.2
- new net 3V3_SENSE: J9.1 (Pin_1)
- new net ACT1_OA1: J4.A1 (Pin_5), J9.9 (Pin_9)
- new net ACT1_OA2: J4.A2 (Pin_6), J9.10 (Pin_10)
- new net ACT1_OB1: J4.B1 (Pin_4), J9.11 (Pin_11)
- new net ACT1_OB2: J4.B2 (Pin_3), J9.12 (Pin_12)
- new net ACT2_OA1: J6.A1 (Pin_5), J9.13 (Pin_13)
- new net ACT2_OA2: J6.A2 (Pin_6), J9.14 (Pin_14)
- new net ACT2_OB1: J6.B1 (Pin_4), J9.15 (Pin_15)
- new net ACT2_OB2: J6.B2 (Pin_3), J9.16 (Pin_16)
- new net ACT3_OA1: J8.A1 (Pin_5), J9.17 (Pin_17)
- new net ACT3_OA2: J8.A2 (Pin_6), J9.18 (Pin_18)
- new net ACT3_OB1: J8.B1 (Pin_4), J9.19 (Pin_19)
- new net ACT3_OB2: J8.B2 (Pin_3), J9.20 (Pin_20)
- new net BAT_GND: C1.2, J12.- (Pin_1), J14.- (Pin_1)
- new net FSR1: J9.5 (Pin_5), R1.1, R2.1
- new net FSR2: J9.6 (Pin_6), R3.1, R4.1
- new net FSR3: J9.7 (Pin_7), R5.1, R6.1
- new net FSR4: J9.8 (Pin_8), R7.1, R8.1
- new net GND: C10.2, C11.2, C12.2, C13.2, C14.2, C15.2, C16.2, C17.2, C18.2, C19.2, C2.2, C20.2, C3.2, C4.2, C5.1, C6.1, C7.2, C8.2, C9.2, J10.GND (Pin_1), J16.- (Pin_1), J2.GND (Pin_9), J4.GND (Pin_7), J6.GND (Pin_7), J8.GND (Pin_7), J9.3 (Pin_3), J9.4 (Pin_4), R10.1, R2.2, R3.2, R5.2, R7.2, SW2.2
- new net VBAT_PRESWITCH: J11.+ (Pin_1), SW1.1
Other:
- note added: "20 PIN CONNECTOR"
- note added: "3.7V 1600MAH BATTERY"
- note added: "BUTTON / SWITCH"
- note added: "ESP32C6 HEADERS"
- note added: "FSR CIRCUIT"
- note added: "GPIO5 uses INPUT_PULLDOWN No external resistor"
- note added: "OLED"
- note added: "Pumped Up Kicks Schematic"
- note added: "TMC2209 HEADERS"
- note added: "VBAT SENSE CIRCUIT"
- note added: "XL6009 BOOST CONVERTER"
- note removed: "4-pin header J_OLED: Pin1: VCC <- 3V3 Pin2: GND Pin3: SDA <- OLED_SDA (GPIO22) Pin4: SCL <- OLED_SCL (GPIO23) I2C address: 0x3C (verify on module) Keep traces short, away from boost zone"
- note removed: "BLOCK 1 - POWER INPUT / BATTERY"
- note removed: "BLOCK 2 - BOOST CONVERTER (XL6009)"
- note removed: "BLOCK 3 - ESP32-C6 SUPERMINI HEADER"
- note removed: "BLOCK 4A - TMC2209 #1 (ACT1)"
- note removed: "BLOCK 4B - TMC2209 #2 (ACT2)"
- note removed: "BLOCK 4C - TMC2209 #3 (ACT3)"
- note removed: "BLOCK 5 - FSR ANALOG FRONT-END x4"
- note removed: "BLOCK 6 - VBAT SENSE"
- note removed: "BLOCK 7 - OLED DISPLAY (SSD1306 0.91")"
- note removed: "BLOCK 8 - USER INTERFACE"
- note removed: "BLOCK 9 - J_MAIN (20-PIN INSOLE CONNECTOR)"
- note removed: "GPIO0 = FSR1_METATARSAL (ADC) GPIO1 = FSR2_ARCH (ADC) GPIO2 = FSR3_CALCANEUS (ADC) GPIO3 = FSR4_AUX (ADC) GPIO4 = STEPPER_ENN (active LOW) GPIO5 = VBAT_SENSE (ADC - 1:2 divider) GPIO6 = ACT1_STEP GPIO7 = ACT1_DIR GPIO9 = CONN_DETECT (INPUT_PULLDOWN) GPIO12 = ACT2_STEP GPIO13 = ACT2_DIR GPIO14 = MODE_BUTTON (INPUT_PULLUP) GPIO20 = ACT3_STEP GPIO21 = ACT3_DIR GPIO22 = OLED_SDA GPIO23 = OLED_SCL AVO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"
- note removed: "LiPo 2-pin connector Main latching power switch TP4056 module 4-pin header VBAT net output to Block 2 USB detect optional Note: charging and actuation MUTUALLY EXCLUSIVE"
- note removed: "Mode button (momentary NO): GPIO14 -- BTN -- GND GPIO14 = INPUT_PULLUP Optional: 100nF across button Connector detect: J_MAIN pin1 (3V3_SENSE) -- 10k --> GPIO9 (INPUT_PULLDOWN) Plugged=HIGH, Removed=LOW Main power switch: Hardware latching switch in series with LiPo -> TP4056 - no GPIO needed"
- note removed: "PIN MAP - DO NOT CHANGE WITHOUT LAYOUT REVIEW"
- note removed: "Per channel FSR1-FSR4: 3V3 | FSR (off-board via J_MAIN pins 5-8) | +-- R_S = 1k --> FSRx_ADC (GPIOx) | | R_D = 10k C=100nF -> GND | GND FSR1 J_MAIN pin5 -> GPIO0 FSR2 J_MAIN pin6 -> GPIO1 FSR3 J_MAIN pin7 -> GPIO2 FSR4 J_MAIN pin8 -> GPIO3 All FSR supply from 3V3 ONLY"
- note removed: "Pin Net Dir 1 3V3_SENSE -> insole (connector detect) 2 5V_SYS -> insole 3 GND 4 GND (duplicate return) 5 FSR1_RAW <- sensor 6 FSR2_RAW <- sensor 7 FSR3_RAW <- sensor 8 FSR4_RAW <- sensor 9 ACT1_OA1 -> coil 10 ACT1_OA2 -> coil 11 ACT1_OB1 -> coil 12 ACT1_OB2 -> coil 13 ACT2_OA1 -> coil 14 ACT2_OA2 -> coil 15 ACT2_OB1 -> coil 16 ACT2_OB2 -> coil 17 ACT3_OA1 -> coil 18 ACT3_OA2 -> coil 19 ACT3_OB1 -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"
- note removed: "Power: VIN <- 5V_SYS GND Output: 3V3 -> 3V3 net GPIO0 FSR1_ADC GPIO1 FSR2_ADC GPIO2 FSR3_ADC GPIO3 FSR4_ADC GPIO4 STEPPER_ENN GPIO5 VBAT_SENSE GPIO6 ACT1_STEP GPIO7 ACT1_DIR GPIO9 CONN_DETECT GPIO12 ACT2_STEP GPIO13 ACT2_DIR GPIO14 MODE_BTN GPIO20 ACT3_STEP GPIO21 ACT3_DIR GPIO22 OLED_SDA GPIO23 OLED_SCL AVOID: GPIO8, GPIO10, GPIO11, GPIO15, USB"
- note removed: "VBAT -- R1=100k --+-- VBAT_SENSE -> GPIO5 | R2=100k | GND Firmware: ADC reads ~VBAT/2, scales x2 < 3.5V = warn < 3.35V = disable motors < 3.2V = shutdown"
- note removed: "VM <- 5V_SYS C_VM = 100uF + 100nF VIO <- 3V3 C_VIO = 100nF GND STEP <- ACT1_STEP DIR <- ACT1_DIR ENN <- STEPPER_ENN OA1/OA2 -> ACT1 coil A -> J_MAIN 9/10 OB1/OB2 -> ACT1 coil B -> J_MAIN 11/12 Test pads: PDN_UART, DIAG"
- note removed: "VM <- 5V_SYS C_VM = 100uF + 100nF VIO <- 3V3 C_VIO = 100nF GND STEP <- ACT2_STEP DIR <- ACT2_DIR ENN <- STEPPER_ENN OA1/OA2 -> ACT2 coil A -> J_MAIN 13/14 OB1/OB2 -> ACT2 coil B -> J_MAIN 15/16 Test pads: PDN_UART, DIAG"
- note removed: "VM <- 5V_SYS C_VM = 100uF + 100nF VIO <- 3V3 C_VIO = 100nF GND STEP <- ACT3_STEP DIR <- ACT3_DIR ENN <- STEPPER_ENN OA1/OA2 -> ACT3 coil A -> J_MAIN 17/18 OB1/OB2 -> ACT3 coil B -> J_MAIN 19/20 Test pads: PDN_UART, DIAG"
- note removed: "XL6009 module 4-pin header Input: VBAT Output: 5V_SYS C_bulk1 = 470uF 35V electrolytic C_bulk2 = 470-1000uF 35V electrolytic C_dec = 100nF ceramic Keep far from FSR analog zone"
